Commit message: Slightly re-factored URDF reading, added Fanuc robot

File: urdfs/fanuc_lrmate200id.urdf (robot description, URDF)
Before this commit: robot fanuc_lrmate200id, 10 links, 9 joints
Links:
- removed link base
- removed link flange
- removed link link_1
- removed link link_2
- removed link link_3
- removed link link_4
- removed link link_5
- removed link link_6
- removed link tool0
- added link Part2, mass 4.85331; collision mesh filename=package://fanuc_motoman/meshes/Part 2.STL scale=0.001 0.001 0.001; visual mesh filename=package://fanuc_motoman/meshes/Part 2.STL scale=0.001 0.001 0.001
- added link Part3, mass 7.96646; collision mesh filename=package://fanuc_motoman/meshes/Part 3.STL scale=0.001 0.001 0.001; visual mesh filename=package://fanuc_motoman/meshes/Part 3.STL scale=0.001 0.001 0.001
- added link Part4, mass 2.401; collision mesh filename=package://fanuc_motoman/meshes/Part 4.STL scale=0.001 0.001 0.001; visual mesh filename=package://fanuc_motoman/meshes/Part 4.STL scale=0.001 0.001 0.001
- added link Part5, mass 2.89084; collision mesh filename=package://fanuc_motoman/meshes/Part 5.STL scale=0.001 0.001 0.001; visual mesh filename=package://fanuc_motoman/meshes/Part 5.STL scale=0.001 0.001 0.001
- added link Part6, mass 0.043284; collision mesh filename=package://fanuc_motoman/meshes/Part 6.STL scale=0.001 0.001 0.001; visual mesh filename=package://fanuc_motoman/meshes/Part 6.STL scale=0.001 0.001 0.001
- added link world
- link base_link: mass None -> 4.85331; geometry collision mesh filename=package://fanuc_motoman/meshes/Part 1.STL scale=0.001 0.001 0.001; visual mesh filename=package://fanuc_motoman/meshes/Part 1.STL scale=0.001 0.001 0.001
Joints:
- removed joint base_link-base
- removed joint joint_1
- removed joint joint_2
- removed joint joint_3
- removed joint joint_4
- removed joint joint_5
- removed joint joint_6
- removed joint joint_6-flange
- removed joint link_6-tool0
- added joint Base_Part2: type continuous, parent base_link, child Part2, origin xyz=0.105 0.09 0.16859, axis 0 0 1
- added joint Part2_Part3: type continuous, parent Part2, child Part3, origin xyz=0.05085 0.0 0.16872 rpy=0 0 0, axis 0 1 0
- added joint Part3_Part4: type continuous, parent Part3, child Part4, origin xyz=0 0 0.44 rpy=0 0 0, axis 0 1 0
- added joint Part4_Part5: type continuous, parent Part4, child Part5, origin xyz=0.1 0 0.025 rpy=0 0 0, axis 1 0 0
- added joint Part6_Part6: type continuous, parent Part5, child Part6, origin xyz=0.325 0 0 rpy=0 0 0, axis 0 1 0
- added joint world_base_joint: type fixed, parent world, child base_link, origin xyz=0 0 0 rpy=0 0 0
