Commit message: Remove unnecessary URDF file.

File: urdfs/vision60.urdf (robot description, URDF)
Before this commit: robot ngr, 17 links, 16 joints
Links:
- removed link toe0
- removed link toe1
- removed link toe2
- removed link toe3
- link hip0: geometry collision box size=0.195 0.17 0.1; visual box size=0.195 0.17 0.1
- link hip1: geometry collision box size=0.195 0.17 0.1; visual box size=0.195 0.17 0.1
- link hip2: geometry collision box size=0.195 0.17 0.1; visual box size=0.195 0.17 0.1
- link hip3: geometry collision box size=0.195 0.17 0.1; visual box size=0.195 0.17 0.1
- link lower0: geometry collision cylinder length=0.28 radius=0.011; collision sphere radius=0.011
- link lower1: geometry collision cylinder length=0.28 radius=0.011; collision sphere radius=0.011
- link lower2: geometry collision cylinder length=0.28 radius=0.011; collision sphere radius=0.011
- link lower3: geometry collision cylinder length=0.28 radius=0.011; collision sphere radius=0.011
Joints:
- removed joint jtoe0
- removed joint jtoe1
- removed joint jtoe2
- removed joint jtoe3
- joint 0: limit lower=-3.14159265359 upper=3.14159265359 effort=87.5 velocity=30 -> (none); origin xyz=0 0.068 0 -> xyz=-.0975 0 0 rpy=0 -0.5 0; type revolute -> continuous
- joint 1: limit lower=0 upper=3.14159265359 effort=87.5 velocity=30 -> (none); origin xyz=-0.25 0 0 -> xyz=-0.25 0 0 rpy=0 0.76 0; type revolute -> continuous
- joint 10: limit lower=-0.43 upper=0.43 effort=375 velocity=8.6 -> (none); type revolute -> continuous
- joint 11: limit lower=-0.43 upper=0.43 effort=375 velocity=8.6 -> (none); type revolute -> continuous
- joint 2: limit lower=-3.14159265359 upper=3.14159265359 effort=87.5 velocity=30 -> (none); origin xyz=0 0.068 0 -> xyz=-.0975 0 0 rpy=0 -0.5 0; type revolute -> continuous
- joint 3: limit lower=0 upper=3.14159265359 effort=87.5 velocity=30 -> (none); origin xyz=-0.25 0 0 -> xyz=-0.25 0 0 rpy=0 0.76 0; type revolute -> continuous
- joint 4: limit lower=-3.14159265359 upper=3.14159265359 effort=87.5 velocity=30 -> (none); origin xyz=0 -0.068 0 -> xyz=-.0975 0 0 rpy=0 -0.5 0; type revolute -> continuous
- joint 5: limit lower=0 upper=3.14159265359 effort=87.5 velocity=30 -> (none); origin xyz=-0.25 0 0 -> xyz=-0.25 0 0 rpy=0 0.76 0; type revolute -> continuous
- joint 6: limit lower=-3.14159265359 upper=3.14159265359 effort=87.5 velocity=30 -> (none); origin xyz=0 -0.068 0 -> xyz=-.0975 0 0 rpy=0 -0.5 0; type revolute -> continuous
- joint 7: limit lower=0 upper=3.14159265359 effort=87.5 velocity=30 -> (none); origin xyz=-0.25 0 0 -> xyz=-0.25 0 0 rpy=0 0.76 0; type revolute -> continuous
- joint 8: limit lower=-0.43 upper=0.43 effort=375 velocity=8.6 -> (none); type revolute -> continuous
- joint 9: limit lower=-0.43 upper=0.43 effort=375 velocity=8.6 -> (none); type revolute -> continuous
