Commit message: added quad climbing robot

File: urdfs/quad_climb_robot.urdf (robot description, URDF)
Before this commit: robot ngr_simple, 13 links, 12 joints
Links:
- added link grab0, mass 0.2; collision sphere radius=0.02; visual sphere radius=0.02
- added link grab1, mass 0.2; collision sphere radius=0.02; visual sphere radius=0.02
- added link grab2, mass 0.2; collision sphere radius=0.02; visual sphere radius=0.02
- added link grab3, mass 0.2; collision sphere radius=0.02; visual sphere radius=0.02
- link body: geometry collision box size=0.3 0.3 0.1; visual box size=0.3 0.3 0.1
- link hip0: geometry collision sphere radius=0.05; visual sphere radius=0.05
- link hip1: geometry collision sphere radius=0.05; visual sphere radius=0.05
- link hip2: geometry collision sphere radius=0.05; visual sphere radius=0.05
- link hip3: geometry collision sphere radius=0.05; visual sphere radius=0.05
- link upper0: geometry collision box size=0.3 0.05 0.05; visual box size=0.3 0.05 0.05
- link upper1: geometry collision box size=0.3 0.05 0.05; visual box size=0.3 0.05 0.05
- link upper2: geometry collision box size=0.3 0.05 0.05; visual box size=0.3 0.05 0.05
- link upper3: geometry collision box size=0.3 0.05 0.05; visual box size=0.3 0.05 0.05
Joints:
- added joint 12: type fixed, parent lower0, child grab0, origin xyz=-0.28 0 0 rpy=0 0 0, axis 1 0 0
- added joint 13: type fixed, parent lower1, child grab1, origin xyz=-0.28 0 0 rpy=0 0 0, axis 1 0 0
- added joint 14: type fixed, parent lower2, child grab2, origin xyz=-0.28 0 0 rpy=0 0 0, axis 1 0 0
- added joint 15: type fixed, parent lower3, child grab3, origin xyz=-0.28 0 0 rpy=0 0 0, axis 1 0 0
- joint 0: axis 0 -1 0 -> 0 1 0; origin xyz=-.0975 0 0 rpy=0 -0.5 0 -> xyz=0 0 0 rpy=0 0.7075 3.14159
- joint 1: origin xyz=-0.25 0 0 rpy=0 0.76 0 -> xyz=-0.28 0 0 rpy=0 -1.57 0
- joint 10: axis 1 0 0 -> 0 0 1; origin xyz=0.325 -0.1575 0 -> xyz=0.15 -0.15 0 rpy=0 0 -0.7075
- joint 11: axis 1 0 0 -> 0 0 1; origin xyz=-0.325 -0.1575 0 -> xyz=-0.15 -0.15 0 rpy=0 0 0.7075
- joint 2: axis 0 -1 0 -> 0 1 0; origin xyz=-.0975 0 0 rpy=0 -0.5 0 -> xyz=0 0 0 rpy=0 0.7075 0
- joint 3: origin xyz=-0.25 0 0 rpy=0 0.76 0 -> xyz=-0.28 0 0 rpy=0 -1.57 0
- joint 4: axis 0 -1 0 -> 0 1 0; origin xyz=-.0975 0 0 rpy=0 -0.5 0 -> xyz=0 0 0 rpy=0 0.7075 3.14159
- joint 5: origin xyz=-0.25 0 0 rpy=0 0.76 0 -> xyz=-0.28 0 0 rpy=0 -1.57 0
- joint 6: axis 0 -1 0 -> 0 1 0; origin xyz=-.0975 0 0 rpy=0 -0.5 0 -> xyz=0 0 0 rpy=0 0.7075 0
- joint 7: origin xyz=-0.25 0 0 rpy=0 0.76 0 -> xyz=-0.28 0 0 rpy=0 -1.57 0
- joint 8: axis 1 0 0 -> 0 0 1; origin xyz=0.325 0.1575 0 -> xyz=0.15 0.15 0 rpy=0 0 0.7075
- joint 9: axis 1 0 0 -> 0 0 1; origin xyz=-0.325 0.1575 0 -> xyz=-0.15 0.15 0 rpy=0 0 -0.7075

Commit message: change fixed joints to revolute.

File: urdfs/quad_climb_robot.urdf (robot description, URDF)
Before this commit: robot ngr_simple, 17 links, 16 joints
Joints:
- joint 12: limit (none) -> lower=0 upper=1.57 effort=100 velocity=30; type fixed -> revolute
- joint 13: limit (none) -> lower=0 upper=1.57 effort=100 velocity=30; type fixed -> revolute
- joint 14: limit (none) -> lower=0 upper=1.57 effort=100 velocity=30; type fixed -> revolute
- joint 15: limit (none) -> lower=0 upper=1.57 effort=100 velocity=30; type fixed -> revolute
