Commit message: Write tests for new LinkJoint constructor. Implement LinkJoint constructor that computes rest transform and screw axis from urdf::JointSharedPtr, the parent link, and the child link

File: urdfs/test/simple_urdf.urdf (robot description, URDF)
Before this commit: robot floating_base_test, 2 links, 1 joints
Joints:
- joint j1: axis (none) -> 1 0 0; limit lower=-0.38 upper=0 effort=1000.0 velocity=0.5 -> lower=-1.57 upper=1.57 effort=1000.0 velocity=0.5; origin (none) -> xyz=0 0 2 rpy=0 0 0
