Commit message: Add test for UniversalRobot four bar linkage. Remove unnecessary code from UniversalRobot class. Fix small error in four bar linkage urdf.

File: urdfs/test/four_bar_linkage.urdf (robot description, URDF)
Before this commit: robot four_bar_linkage, 5 links, 5 joints
Joints:
- joint j4: origin xyz=0 0 0 rpy=1.57079632679 0 0 -> xyz=0 0 2 rpy=1.57079632679 0 0
