Commit message: improve visualization by adding locations

File: urdfs/test/four_bar_linkage_pure.urdf (robot description, URDF)
Before this commit: robot four_bar_linkage, 4 links, 4 joints
Links:
- link l2: mass 15 -> 100
- link l3: mass 15 -> 11005

Commit message: revised error in screw axis, four bar linkage test pass

File: urdfs/test/four_bar_linkage_pure.urdf (robot description, URDF)
Before this commit: robot four_bar_linkage, 4 links, 4 joints
Links:
- link l1: mass 100 -> 1
- link l2: mass 100 -> 1
- link l3: mass 11005 -> 1
- link l4: mass 100 -> 1

Commit message: Removed URDF parsing submodules
Eliminate urdfdom dependency and transition solely to sdformat.

Remove urdfdom urdfdom_headers files

Remove urdfdom/urdfdom_headers dependencies. Transition solely to
sdformat.

File: urdfs/test/four_bar_linkage_pure.urdf (robot description, URDF)
Before this commit: robot four_bar_linkage, 4 links, 4 joints
Links:
- link l1: geometry visual cylinder length=2 radius=0.2
- link l2: geometry visual cylinder length=2 radius=0.2
- link l3: geometry visual cylinder length=2 radius=0.2
- link l4: geometry visual cylinder length=2 radius=0.2
