Commit message: # Conflicts: #	gtdynamics/kinematics/Kinematics.h #	gtdynamics/kinematics/KinematicsInterval.cpp #	gtdynamics/kinematics/KinematicsSlice.cpp #	gtdynamics/kinematics/KinematicsTrajectory.cpp #	gtdynamics/pandarobot/gpmp/GaussianProcessPrior.h #	gtdynamics/universal_robot/Joint.cpp

File: models/urdfs/cart_pole.urdf (robot description, URDF)
Before this commit: robot cart_pole, 3 links, 2 joints
Joints:
- joint j1: origin xyz=0 0 0 rpy=3.1415 0 0 -> xyz=0 0 0 rpy=3.141592653589793238 0 0
